Commit message: urdfをlaunchで確認できるようにした

File: urdf/robovie.urdf (robot description, URDF)
Before this commit: robot robovie, 8 links, 7 joints
Links:
- removed link left_arm_link1
- removed link left_arm_link2
- removed link left_arm_link3
- removed link right_arm_link1
- removed link right_arm_link2
- removed link right_arm_link3
- added link left_arm_link_1
- added link left_arm_link_2
- added link left_elbow_link
- added link left_shoulder_link
- added link right_arm_link_1
- added link right_arm_link_2
- added link right_elbow_link
- added link right_shoulder_link
Joints:
- removed joint left_elbow
- removed joint left_shoulder
- removed joint left_wrist
- removed joint neck_joint
- removed joint right_elbow
- removed joint right_shoulder
- removed joint right_wrist
- added joint left_elbow_pitch: type revolute, parent left_arm_link_1, child left_elbow_link, origin xyz=0 0.11 0 rpy=0 0 0, axis 0 1 0, limit lower=-1.57 upper=1.57 effort=0.5293 velocity=6.159937255
- added joint left_elbow_roll: type revolute, parent left_elbow_link, child left_arm_link_2, origin xyz=0 0 0 rpy=0 0 0, axis 1 0 0, limit lower=-2.0944 upper=0 effort=0.5293 velocity=6.159937255
- added joint left_shoulder_pitch: type revolute, parent shoulder_link, child left_shoulder_link, origin xyz=0 -0.19 0 rpy=0 0 0, axis 0 1 0, limit lower=-1.57 upper=3.14 effort=0.5293 velocity=6.159937255
- added joint left_shoulder_roll: type revolute, parent left_shoulder_link, child left_arm_link_1, origin xyz=0 0 0 rpy=0 0 0, axis -1 0 0, limit lower=-1.57 upper=1.39626 effort=0.5293 velocity=6.159937255
- added joint right_elbow_pitch: type revolute, parent right_arm_link_1, child right_elbow_link, origin xyz=0 0.11 0 rpy=0 0 0, axis 0 1 0, limit lower=-1.57 upper=1.57 effort=0.5293 velocity=6.159937255
- added joint right_elbow_roll: type revolute, parent right_elbow_link, child right_arm_link_2, origin xyz=0 0 0 rpy=0 0 0, axis 1 0 0, limit lower=-2.0944 upper=0 effort=0.5293 velocity=6.159937255
- added joint right_shoulder_pitch: type revolute, parent shoulder_link, child right_shoulder_link, origin xyz=0 0.19 0 rpy=0 0 0, axis 0 1 0, limit lower=-1.57 upper=3.14 effort=0.5293 velocity=6.159937255
- added joint right_shoulder_roll: type revolute, parent right_shoulder_link, child right_arm_link_1, origin xyz=0 0 0 rpy=0 0 0, axis 1 0 0, limit lower=-1.57 upper=1.39626 effort=0.5293 velocity=6.159937255
- added joint shoulder_joint: type fixed, parent base_link, child shoulder_link, origin xyz=0 0 0.71 rpy=0 0 0

Commit message: rad -> target変換式修正

File: urdf/robovie.urdf (robot description, URDF)
Before this commit: robot robovie, 10 links, 9 joints
Joints:
- joint left_elbow_pitch: origin xyz=0 0.11 0 rpy=0 0 0 -> xyz=0 0.11 0 rpy=0 1.57 0
- joint left_elbow_roll: limit lower=-2.0944 upper=0 effort=0.5293 velocity=6.159937255 -> lower=3.14 upper=5.236 effort=0.5293 velocity=6.159937255; origin xyz=0 0 0 rpy=0 0 0 -> xyz=0 0 0 rpy=3.14 -1.57 0
- joint left_shoulder_roll: limit lower=-1.57 upper=1.39626 effort=0.5293 velocity=6.159937255 -> lower=1.57 upper=4.53786 effort=0.5293 velocity=6.159937255
