Commit message: 座標系が鏡なのを修正

File: urdf/robovie_rotated.urdf (robot description, URDF)
Before this commit: robot robovie, 10 links, 9 joints
Joints:
- joint left_elbow_roll: axis -1 0 0 -> 1 0 0
- joint left_shoulder_pitch: origin xyz=0 0.19 0 rpy=0 0 0 -> xyz=0 -0.19 0 rpy=0 0 0
- joint left_shoulder_roll: axis 1 0 0 -> -1 0 0; limit lower=4.71293 upper=7.67945 effort=0.5293 velocity=6.159937255 -> lower=1.57 upper=4.53786 effort=0.5293 velocity=6.159937255
- joint right_elbow_roll: axis -1 0 0 -> 1 0 0; limit lower=0 upper=1.57 effort=0.5293 velocity=6.159937255 -> lower=-2.0944 upper=0 effort=0.5293 velocity=6.159937255
- joint right_shoulder_pitch: axis 0 -1 0 -> 0 1 0; limit lower=-3.14 upper=1.57 effort=0.5293 velocity=6.159937255 -> lower=-1.57 upper=3.14 effort=0.5293 velocity=6.159937255; origin xyz=0 -0.19 0 rpy=0 0 0 -> xyz=0 0.19 0 rpy=0 0 0
- joint right_shoulder_roll: limit lower=1.74533 upper=4.71239 effort=0.5293 velocity=6.159937255 -> lower=-1.57 upper=1.39626 effort=0.5293 velocity=6.159937255
